File: pcb 5-3/pcb.kicad_pcb (KiCad board)
At the start: 2 copper layers, 14 parts, among them J1 Conn_01x10_Pin, J2 Conn_01x04_Socket, U1 MQ-6, U2 MQ-6, U3 MQ-6, U4 MQ-6

Commit message: Fixed "PCB Fixes (URGENT) #1"
Other:
- board outline added: 127.5 x 34.5 mm
Changed lines of the file:
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@@
 			(outputformat 1)
 			(mirror no)
-			(drillshape 1)
+			(drillshape 0)
 			(scaleselection 1)
-			(outputdirectory "")
+			(outputdirectory "C:/Users/mikey/Downloads/export/")
 		)
 	)
@@
 		)
 	)
+	(gr_rect
+		(start 77.5 31.5)
+		(end 205 66)
+		(stroke
+			(width 0.05)
+			(type default)
+		)
+		(fill none)
+		(layer "Edge.Cuts")
+	)
 	(segment
 		(start 176.9125 54.5875)
@@
 		(polygon
 			(pts
-				(xy 124.202728 54.27977) (xy 125 45) (xy 125 44) (xy 115 44) (xy 115 47) (xy 122 47) (xy 122 55.5)
+				(xy 124.5 51.5) (xy 124.968965 47.046653) (xy 125 44) (xy 115 44) (xy 115 47) (xy 122 47) (xy 122 55.5)
 				(xy 124 55.5)
 			)
@@
 		(polygon
 			(pts
-				(xy 139.5 46.5) (xy 147 46.5) (xy 147 55.5) (xy 148.5 55.5) (xy 148.5 43.5) (xy 139.5 43.5)
+				(xy 139.5 46.5) (xy 147 46.5) (xy 147 55.5) (xy 149 51.5) (xy 149 43.5) (xy 139.5 43.5)
 			)
 		)
@@
 		(polygon
 			(pts
-				(xy 162.5 46.5) (xy 170 46.5) (xy 170 55.5) (xy 171.5 55.5) (xy 171.5 43.5) (xy 162.5 43.5)
+				(xy 162.5 46.5) (xy 169.5 46.5) (xy 169.5 56) (xy 171.516313 55.98377) (xy 172.016313 43.48377)
+				(xy 162.5 43.5)
 			)
 		)
